File: minicurso.sch (KiCad schematic (older format))
At the start: 5 parts

Commit message: Footprints selecionadas
Parts:
- C1: renamed from C?; footprint (none) -> Capacitor_THT:C_Disc_D3.0mm_W2.0mm_P2.50mm
- R1, R2, R3: renamed from R?; footprint (none) -> Resistor_THT:R_Axial_DIN0204_L3.6mm_D1.6mm_P7.62mm_Horizontal
- gave numbers to parts that had none: 1
Changed lines of the file:
@@
 $EndDescr
 $Comp
-L Device:R_Small R?
+L Device:R_Small R1
 U 1 1 5D4E527F
 P 2100 3600
-F 0 "R?" V 1904 3600 50  0000 C CNN
+F 0 "R1" V 1904 3600 50  0000 C CNN
 F 1 "1k" V 1995 3600 50  0000 C CNN
-F 2 "" H 2100 3600 50  0001 C CNN
+F 2 "Resistor_THT:R_Axial_DIN0204_L3.6mm_D1.6mm_P7.62mm_Horizontal" H 2100 3600 50  0001 C CNN
 F 3 "~" H 2100 3600 50  0001 C CNN
 	1    2100 3600
@@
 $EndComp
 $Comp
-L Device:R_Small R?
+L Device:R_Small R2
 U 1 1 5D4E5811
 P 2350 3850
-F 0 "R?" H 2409 3896 50  0000 L CNN
+F 0 "R2" H 2409 3896 50  0000 L CNN
 F 1 "510k" H 2409 3805 50  0000 L CNN
-F 2 "" H 2350 3850 50  0001 C CNN
+F 2 "Resistor_THT:R_Axial_DIN0204_L3.6mm_D1.6mm_P7.62mm_Horizontal" H 2350 3850 50  0001 C CNN
 F 3 "~" H 2350 3850 50  0001 C CNN
 	1    2350 3850
@@
 $EndComp
 $Comp
-L Device:R_Small R?
+L Device:R_Small R3
 U 1 1 5D4E5B79
 P 2800 4050
-F 0 "R?" H 2859 4096 50  0000 L CNN
+F 0 "R3" H 2859 4096 50  0000 L CNN
 F 1 "10k" H 2859 4005 50  0000 L CNN
-F 2 "" H 2800 4050 50  0001 C CNN
+F 2 "Resistor_THT:R_Axial_DIN0204_L3.6mm_D1.6mm_P7.62mm_Horizontal" H 2800 4050 50  0001 C CNN
 F 3 "~" H 2800 4050 50  0001 C CNN
 	1    2800 4050
@@
 $EndComp
 $Comp
-L Device:C_Small C?
+L Device:C_Small C1
 U 1 1 5D4E6120
 P 1650 3600
-F 0 "C?" V 1421 3600 50  0000 C CNN
+F 0 "C1" V 1421 3600 50  0000 C CNN
 F 1 "20nF" V 1512 3600 50  0000 C CNN
-F 2 "" H 1650 3600 50  0001 C CNN
+F 2 "Capacitor_THT:C_Disc_D3.0mm_W2.0mm_P2.50mm" H 1650 3600 50  0001 C CNN
 F 3 "~" H 1650 3600 50  0001 C CNN
 	1    1650 3600
@@
 $EndComp
 $Comp
-L Transistor_BJT:BC548 Q?
+L Transistor_BJT:BC548 Q1
 U 1 1 5D4E6C54
 P 2700 3600
-F 0 "Q?" H 2891 3646 50  0000 L CNN
+F 0 "Q1" H 2891 3646 50  0000 L CNN
 F 1 "BC548" H 2891 3555 50  0000 L CNN
 F 2 "Package_TO_SOT_THT:TO-92_Inline" H 2900 3525 50  0001 L CIN
@@
 $EndComp
 $Comp
-L power:GND #PWR?
+L power:GND #PWR0101
 U 1 1 5D4E7D4F
 P 2800 4300
-F 0 "#PWR?" H 2800 4050 50  0001 C CNN
+F 0 "#PWR0101" H 2800 4050 50  0001 C CNN
 F 1 "GND" H 2805 4127 50  0000 C CNN
 F 2 "" H 2800 4300 50  0001 C CNN
@@
 $EndComp
 $Comp
-L power:VCC #PWR?
+L power:VCC #PWR0102
 U 1 1 5D4E8678
 P 2800 3200
-F 0 "#PWR?" H 2800 3050 50  0001 C CNN
+F 0 "#PWR0102" H 2800 3050 50  0001 C CNN
 F 1 "VCC" H 2817 3373 50  0000 C CNN
 F 2 "" H 2800 3200 50  0001 C CNN
@@
 	2800 4150 2800 4300
 $Comp
-L power:GND #PWR?
+L power:GND #PWR0103
 U 1 1 5D4EA4D1
 P 2350 4100
-F 0 "#PWR?" H 2350 3850 50  0001 C CNN
+F 0 "#PWR0103" H 2350 3850 50  0001 C CNN
 F 1 "GND" H 2355 3927 50  0000 C CNN
 F 2 "" H 2350 4100 50  0001 C CNN
